Commit message: first update

File: husky_description/urdf/decorations.urdf.xacro (robot description, xacro)
@@ -22,11 +22,11 @@
 -->
 <robot name="husky_decorations" xmlns:xacro="http://ros.org/wiki/xacro">
-  <material name="dark_grey"><color rgba="0.2 0.2 0.2 1.0" /></material>
-  <material name="medium_grey"><color rgba="0.6 0.6 0.6 1.0" /></material>
+  <!-- <material name="dark_grey_husky"><color rgba="0.2 0.2 0.2 1.0" /></material> -->
+  <!-- <material name="medium_grey"><color rgba="0.6 0.6 0.6 1.0" /></material>
   <material name="light_grey"><color rgba="0.8 0.8 0.8 1.0" /></material>
   <material name="yellow"><color rgba="0.8 0.8 0.0 1.0" /></material>
   <material name="black"><color rgba="0.15 0.15 0.15 1.0" /></material>
   <material name="white"><color rgba="1.0 1.0 1.0 1.0" /></material>
-  <material name="red"><color rgba="1.0 0.0 0.0 1.0" /></material>
+  <material name="red"><color rgba="1.0 0.0 0.0 1.0" /></material> -->
   <xacro:macro name="husky_decorate">
     <!--
@@ -44,8 +44,8 @@
     <xacro:property name="husky_wibotic_bumper_enable"  value="$(optenv HUSKY_WIBOTIC_BUMPER 0)" />
     <!-- Top Plate -->
-    <xacro:property name="pacs_enable"                  value="$(optenv HUSKY_PACS_ENABLED false)"/>
+    <xacro:property name="pacs_enable"                  value="false"/>
     <xacro:property name="top_plate_enable"             value="$(optenv HUSKY_TOP_PLATE_ENABLED true)"/>
     <xacro:property name="large_top_plate_enable"       value="$(optenv HUSKY_LARGE_TOP_PLATE false)"/>
-    <xacro:property name="user_rail_enable"             value="$(optenv HUSKY_USER_RAIL_ENABLED true)"/>
+    <xacro:property name="user_rail_enable"             value="true"/>
     <!--
       CHASSIS: Spawn and attach default chassis.
@@ -156,5 +156,5 @@
       <!-- Attach user rails to base link -->
       <joint name="user_rail" type="fixed">
-        <origin xyz="0.272 0 0.245" rpy="0 0 0" />
+        <origin xyz="-0.285 0 0.79" rpy="0 -1.57 0" />
         <parent link="base_link" />
         <child link="user_rail_link" />

Commit message: moveit

File: husky_description/urdf/decorations.urdf.xacro (robot description, xacro)
@@ -151,6 +151,13 @@
           <geometry>
             <mesh filename="package://husky_description/meshes/user_rail.dae" />
-          </geometry>
-        </visual>
+            <!-- <box size="0.475 0.423 0.268"/> -->
+          </geometry>
+        </visual>
+        <collision>
+          <origin xyz="-0.3  0.0 0.0" rpy="0 0 0" />
+          <geometry>
+            <box size="0.475 0.423 0.268"/>
+          </geometry>
+        </collision>
       </link>
       <!-- Attach user rails to base link -->
